Commit message: Added in simulation details and plotting abilities

File: src/baxter_simulator/baxter_sim_examples/models/block/model.urdf (robot description, URDF)
Before this commit: robot block, 1 links, 0 joints
Links:
- link block: geometry collision box size=0.05 0.05 0.20; visual box size=0.05 0.05 0.20
